File: hardware/testrack_breakout/testrack_breakout.kicad_sch (KiCad schematic)
At the start: 10 parts, among them J1 USB_C_Receptacle_USB2.0_16P, J2 Conn_02x05_Odd_Even, J3 Conn_02x10_Odd_Even, J4 Conn_01x04, J5 Conn_02x09_Odd_Even

Commit message: Placed and routed the components for the breakout board
Parts:
- added H1, H2, H3, H4: MountingHole_Pad, MountingHole:MountingHole_3.2mm_M3_Pad, symbol Mechanical:MountingHole_Pad
- added H5: MountingHole_Pad, pkl_connectors:M2_MountingPost, symbol Mechanical:MountingHole_Pad
- J2: footprint (none) -> rhais_connector-pinheader:PinHeader_2x05_P1.27mm_Vertical_SMD
- J3: footprint (none) -> Connector_PinHeader_1.27mm:PinHeader_2x10_P1.27mm_Vertical_SMD
- J4: footprint (none) -> Connector_JST:JST_SH_SM04B-SRSS-TB_1x04-1MP_P1.00mm_Horizontal
- J5: footprint (none) -> Connector_PinHeader_2.54mm:PinHeader_2x09_P2.54mm_Vertical
- JP1: footprint (none) -> pkl_connectors:TE_2199230-7_67_P0.5mm_Horizontal; MFR_LCSC (none) -> JAE; MPN_LCSC (none) -> SM3ZS067U410ABR1000; OC_LCSC (none) -> C4730576
- R1, R2: footprint (none) -> rhais_rcl:R0603; MFR_LCSC (none) -> VO; MPN_LCSC (none) -> SCR0603F5K1; OC_LCSC (none) -> C3016319
- R3, R4: footprint (none) -> rhais_rcl:R0603; MFR_FARNELL (none) -> PANASONIC; MFR_LCSC (none) -> PANASONIC; MPN_FARNELL (none) -> ERJU03F2201V; MPN_LCSC (none) -> ERJ-U03F2201V; OC_FARNELL (none) -> 2145349; OC_LCSC (none) -> C1859135
Connections:
- net GND: now also H1.1, H2.1, H3.1, H4.1, H5.1
