File: hardware/testrack_module_stm32h5/testrack_module_stm32h5.kicad_pcb (KiCad board)
At the start: 4 copper layers, 38 x 38 mm, 23 parts, among them U1 STM32H573VITx, U2 24AA01-I/SN, U3 LT1962-3.3, Y1 32.768kHz, Y2 25MHz

Commit message: Variety of fixes for the STM32h5 module
Connections:
- U1 pad 14: /~{RST} -> /NRST
